Commit message: nav2 partial

File: description/gazebo_control.xacro (robot description, xacro)
@@ -17,9 +17,9 @@
          <left_joint>back_left_wheel_joint</left_joint>
          <right_joint>back_right_wheel_joint</right_joint>
-         <wheel_separation>0.66</wheel_separation>
-         <wheel_separation>0.66</wheel_separation>
+         <wheel_separation>0.730</wheel_separation>
+         <wheel_separation>0.730</wheel_separation>
          <wheel_diameter>0.25</wheel_diameter>
          <wheel_diameter>0.25</wheel_diameter>
-         <max_wheel_torque>20</max_wheel_torque>
+         <max_wheel_torque>5</max_wheel_torque>
          <max_wheel_acceleration>1.0</max_wheel_acceleration>
          <publish_odom>true</publish_odom>

File: description/robot.urdf.xacro (robot description, xacro)
@@ -1,5 +1,18 @@
 <?xml version="1.0"?>
 <robot xmlns:xacro="http://www.ros.org/wiki/xacro"  name="robot">
+    <!-- <xacro:arg name="use_ros2_control" default="true"/>
     <xacro:include filename="robot_core.xacro" />
+    <xacro:if value="$(arg use_ros2_control)">
+        <xacro:include filename="ros2_control.xacro" />
+    </xacro:if>
+    <xacro:unless value="$(arg use_ros2_control)">
+        <xacro:include filename="gazebo_control.xacro" />
+    </xacro:unless>
+    <xacro:include filename="gps.xacro" />
+    <xacro:include filename="imu.xacro" /> -->
+    <!-- <xacro:include filename="lidar.xacro" /> -->
+    <!-- <xacro:include filename="camera.xacro" /> -->
+    <!-- <xacro:include filename="depth_camera.xacro" /> -->
     <xacro:include filename="gazebo_control.xacro" />
+    <xacro:include filename="URDF.xacro" />
 </robot>

File: description/robot_core.xacro (robot description, xacro)
@@ -14,4 +14,31 @@
         <color rgba="0 0 0 1"/>
     </material>
+    <material name="red">
+        <color rgba="1 0 0 1"/>
+    </material>
+    <!-- <joint name="base_footprint_joint" type="fixed">
+        <parent link="base_link"/>
+        <child link="base_link"/>
+        <origin xyz="0 0 0" rpy="0 0 0"/>
+    </joint>
+    <link name="base_link">
+        <visual>
+      <origin xyz="0 0 0.0" rpy="0 0 0"/>
+      <material name="black"/>
+    </visual> -->
+    <!-- <collision>
+      <origin xyz="0.0 0 0.0" rpy="0 0 0"/>
+      <geometry>
+        <box size="0.3 0.3 0.27"/>
+      </geometry>
+    </collision>
+    <inertial>
+      <origin xyz="0 0 0" rpy="0 0 0"/>
+      <mass value="1.3729096e+00"/>
+      <inertia ixx="8.7002718e-03" ixy="-4.7576583e-05" ixz="1.1160499e-04"
+               iyy="8.6195418e-03" iyz="-3.5422299e-06"
+               izz="1.4612727e-02" />
+    </inertial>
+    </link> -->
     <!-- BASE LINK -->
     <link name="base_link">
@@ -60,5 +87,5 @@
         <collision>
             <geometry>
-                <cylinder radius="0.125" length="0.04"/>
+                <sphere radius="0.125" />
             </geometry>
         </collision>
@@ -86,5 +113,5 @@
         <collision>
             <geometry>
-                <cylinder radius="0.125" length="0.04"/>
+                <sphere radius="0.125" />
             </geometry>
         </collision>
@@ -112,5 +139,5 @@
         <collision>
             <geometry>
-                <cylinder radius="0.125" length="0.4"/>
+                <sphere radius="0.125" />
             </geometry>
         </collision>
@@ -138,5 +165,5 @@
         <collision>
             <geometry>
-                <cylinder radius="0.125" length="0.4"/>
+                <sphere radius="0.125" />
             </geometry>
         </collision>
@@ -148,4 +175,11 @@
         <material>Gazebo/Blue</material>
     </gazebo>
+    <!-- Add the gps link so we get a static transform for the GPS
+    <joint name="gps_joint" type="fixed">
+        <parent link="base_link"/>
+        <child link="gps_link"/>
+        <origin xyz="0 0 0" rpy="0 0 0"/>
+    </joint>
+    <link name="gps_link"/> -->
     <!-- CASTER WHEEL LINK
     <joint name="caster_wheel_joint" type="fixed">

File: install/my_bot/share/my_bot/description/gazebo_control.xacro (robot description, xacro)
@@ -1 +1 @@
-/home/sunil-ubuntu/dev_ws/src/my_bot/description/gazebo_control.xacro
+unsupported reparse point

File: install/my_bot/share/my_bot/description/inertial_macros.xacro (robot description, xacro)
@@ -1 +1 @@
-/home/sunil-ubuntu/dev_ws/src/my_bot/description/inertial_macros.xacro
+unsupported reparse point

File: install/my_bot/share/my_bot/description/robot.urdf.xacro (robot description, xacro)
@@ -1 +1 @@
-/home/sunil-ubuntu/dev_ws/src/my_bot/description/robot.urdf.xacro
+unsupported reparse point

File: install/my_bot/share/my_bot/description/robot_core.xacro (robot description, xacro)
@@ -1 +1 @@
-/home/sunil-ubuntu/dev_ws/src/my_bot/description/robot_core.xacro
+unsupported reparse point
