Commit message: model sdf

File: model/robot/robot_core.xacro (robot description, xacro)
@@ -17,11 +17,28 @@
         <color rgba="1 0 0 1"/>
     </material>
-    <joint name="base_footprint_joint" type="fixed">
-        <parent link="base_link"/>
-        <child link="base_footprint"/>
+    <!-- <joint name="base_footprint_joint" type="fixed">
+        <parent link="base_link"/>
+        <child link="base_link"/>
         <origin xyz="0 0 0" rpy="0 0 0"/>
     </joint>
-    <link name="base_footprint">
-    </link>
+    <link name="base_link">
+        <visual>
+      <origin xyz="0 0 0.0" rpy="0 0 0"/>
+      <material name="black"/>
+    </visual> -->
+    <!-- <collision>
+      <origin xyz="0.0 0 0.0" rpy="0 0 0"/>
+      <geometry>
+        <box size="0.3 0.3 0.27"/>
+      </geometry>
+    </collision>
+    <inertial>
+      <origin xyz="0 0 0" rpy="0 0 0"/>
+      <mass value="1.3729096e+00"/>
+      <inertia ixx="8.7002718e-03" ixy="-4.7576583e-05" ixz="1.1160499e-04"
+               iyy="8.6195418e-03" iyz="-3.5422299e-06"
+               izz="1.4612727e-02" />
+    </inertial>
+    </link> -->
     <!-- BASE LINK -->
     <link name="base_link">
@@ -47,11 +64,20 @@
             </geometry>
         </collision>
-        <xacro:inertial_box mass="0.5" x="0.3" y="0.3" z="0.15">
-            <origin xyz="0.3 0 0.135" rpy="0 0 0"/>
-        </xacro:inertial_box>
-    </link>
-    <gazebo reference="chassis">
+        <inertial>
+			<pose>0.3 0 0.135 0 0 0</pose>
+			<mass>13.4817350958382</mass>
+			<inertia>
+				<ixx>0.314898837628642</ixx>
+				<ixy>-1.83915405182082E-05</ixy>
+				<ixz>9.71911553669445E-05</ixz>
+				<iyy>0.27110302696631</iyy>
+				<iyz>-2.51545485645537E-07</iyz>
+				<izz>0.545868688934175</izz>
+			</inertia>
+	    </inertial>
+    </link>
+    <!-- <gazebo reference="chassis">
         <material>Gazebo/White</material>
-    </gazebo>
+    </gazebo> -->
     <!-- LEFT back WHEEL LINK -->
     <joint name="back_left_wheel_joint" type="continuous">
@@ -158,4 +184,11 @@
         <material>Gazebo/Blue</material>
     </gazebo>
+    <!-- Add the gps link so we get a static transform for the GPS
+    <joint name="gps_joint" type="fixed">
+        <parent link="base_link"/>
+        <child link="gps_link"/>
+        <origin xyz="0 0 0" rpy="0 0 0"/>
+    </joint>
+    <link name="gps_link"/> -->
     <!-- CASTER WHEEL LINK
     <joint name="caster_wheel_joint" type="fixed">

Commit message: basic

File: model/robot/robot_core.xacro (robot description, xacro)
@@ -17,28 +17,11 @@
         <color rgba="1 0 0 1"/>
     </material>
-    <!-- <joint name="base_footprint_joint" type="fixed">
+    <joint name="base_footprint_joint" type="fixed">
         <parent link="base_link"/>
-        <child link="base_link"/>
+        <child link="base_footprint"/>
         <origin xyz="0 0 0" rpy="0 0 0"/>
     </joint>
-    <link name="base_link">
-        <visual>
-      <origin xyz="0 0 0.0" rpy="0 0 0"/>
-      <material name="black"/>
-    </visual> -->
-    <!-- <collision>
-      <origin xyz="0.0 0 0.0" rpy="0 0 0"/>
-      <geometry>
-        <box size="0.3 0.3 0.27"/>
-      </geometry>
-    </collision>
-    <inertial>
-      <origin xyz="0 0 0" rpy="0 0 0"/>
-      <mass value="1.3729096e+00"/>
-      <inertia ixx="8.7002718e-03" ixy="-4.7576583e-05" ixz="1.1160499e-04"
-               iyy="8.6195418e-03" iyz="-3.5422299e-06"
-               izz="1.4612727e-02" />
-    </inertial>
-    </link> -->
+    <link name="base_footprint">
+    </link>
     <!-- BASE LINK -->
     <link name="base_link">
@@ -64,20 +47,11 @@
             </geometry>
         </collision>
-        <inertial>
-			<pose>0.3 0 0.135 0 0 0</pose>
-			<mass>13.4817350958382</mass>
-			<inertia>
-				<ixx>0.314898837628642</ixx>
-				<ixy>-1.83915405182082E-05</ixy>
-				<ixz>9.71911553669445E-05</ixz>
-				<iyy>0.27110302696631</iyy>
-				<iyz>-2.51545485645537E-07</iyz>
-				<izz>0.545868688934175</izz>
-			</inertia>
-	    </inertial>
+        <xacro:inertial_box mass="0.5" x="0.3" y="0.3" z="0.15">
+            <origin xyz="0.3 0 0.135" rpy="0 0 0"/>
+        </xacro:inertial_box>
     </link>
-    <!-- <gazebo reference="chassis">
+    <gazebo reference="chassis">
         <material>Gazebo/White</material>
-    </gazebo> -->
+    </gazebo>
     <!-- LEFT back WHEEL LINK -->
     <joint name="back_left_wheel_joint" type="continuous">
@@ -184,11 +158,4 @@
         <material>Gazebo/Blue</material>
     </gazebo>
-    <!-- Add the gps link so we get a static transform for the GPS
-    <joint name="gps_joint" type="fixed">
-        <parent link="base_link"/>
-        <child link="gps_link"/>
-        <origin xyz="0 0 0" rpy="0 0 0"/>
-    </joint>
-    <link name="gps_link"/> -->
     <!-- CASTER WHEEL LINK
     <joint name="caster_wheel_joint" type="fixed">
